Commit message: Fix finger URDF

File: src/roborscht_description/urdf/finger.urdf (robot description, URDF)
Before this commit: robot finger, 5 links, 4 joints
Links:
- link base_link: mass 0.011452 -> 0.0119128649201374
- link distal_link: mass 0.0032456 -> 0.00324558485631147
- link metacarpal_link: mass 0.0058359 -> 0.00537510095982113
- link middle_link: mass 0.0043864 -> 0.00438641275668905
- link proximal_link: mass 0.0045745 -> 0.00457448104418533
Joints:
- joint distal_joint: axis 1 0 0 -> 0 0 -1; limit lower=0 upper=0.523 effort=0 velocity=0 -> lower=-1.309 upper=0 effort=0 velocity=0; origin xyz=0 0.0010283 0.032416 rpy=-0.063144 0 0 -> xyz=0.033172 0 0 rpy=-3.1416 0 3.0784
- joint metacarpal_joint: axis 0 1 0 -> 0 0 1; limit lower=0 upper=0.523 effort=0 velocity=0 -> lower=-0.2618 upper=0.2618 effort=0 velocity=0; origin xyz=-0.0010929 0.001 0.057418 rpy=0 -0.049938 0 -> xyz=-0.0016899 -0.051494 0.059041 rpy=-1.5708 -0.049938 3.1416
- joint middle_joint: axis 1 0 0 -> 0 0 1; limit lower=0 upper=0.523 effort=0 velocity=0 -> lower=-1.309 upper=0 effort=0 velocity=0; origin xyz=0 0.00018799 0.033414 rpy=-0.011388 0 0 -> xyz=0.033972 0 0 rpy=0 0 -0.011388
- joint proximal_joint: axis 1 0 0 -> 0 0 1; limit lower=0 upper=0.523 effort=0 velocity=0 -> lower=-1.309 upper=0 effort=0 velocity=0; origin xyz=0 -0.0015038 0.034991 rpy=0.085673 0 0 -> xyz=0 -0.038786 -0.007734 rpy=-1.5708 0.085673 -1.5708

Commit message: Create new URDF

File: src/roborscht_description/urdf/finger.urdf (robot description, URDF)
Before this commit: robot finger, 5 links, 4 joints
Joints:
- joint distal_joint: mimic (none) -> joint=middle_joint multiplier=1 offset=0
- joint middle_joint: mimic (none) -> joint=proximal_joint multiplier=1 offset=0
