Commit message: Add tm5x-900 robot arm

File: src/roborscht_description/urdf/roborscht_v2.urdf (robot description, URDF)
Before this commit: robot roborscht_v2, 22 links, 21 joints
Joints:
- joint index_distal_joint: limit lower=-0.698 upper=0 effort=0 velocity=0 -> lower=-1.309 upper=0 effort=0 velocity=0
- joint index_middle_joint: limit lower=-0.698 upper=0 effort=0 velocity=0 -> lower=-1.309 upper=0 effort=0 velocity=0
- joint index_proximal_joint: limit lower=-0.698 upper=0 effort=0 velocity=0 -> lower=-1.309 upper=0 effort=0 velocity=0
- joint little_distal_joint: limit lower=-0.698 upper=0 effort=0 velocity=0 -> lower=-1.309 upper=0 effort=0 velocity=0
- joint little_middle_joint: limit lower=-0.698 upper=0 effort=0 velocity=0 -> lower=-1.309 upper=0 effort=0 velocity=0
- joint little_proximal_joint: limit lower=-0.698 upper=0 effort=0 velocity=0 -> lower=-1.309 upper=0 effort=0 velocity=0
- joint middle_distal_joint: limit lower=-0.698 upper=0 effort=0 velocity=0 -> lower=-1.309 upper=0 effort=0 velocity=0
- joint middle_middle_joint: limit lower=-0.698 upper=0 effort=0 velocity=0 -> lower=-1.309 upper=0 effort=0 velocity=0
- joint middle_proximal_joint: limit lower=-0.698 upper=0 effort=0 velocity=0 -> lower=-1.309 upper=0 effort=0 velocity=0
- joint ring_distal_joint: limit lower=-0.698 upper=0 effort=0 velocity=0 -> lower=-1.309 upper=0 effort=0 velocity=0
- joint ring_middle_joint: limit lower=-0.698 upper=0 effort=0 velocity=0 -> lower=-1.309 upper=0 effort=0 velocity=0
- joint ring_proximal_joint: limit lower=-0.698 upper=0 effort=0 velocity=0 -> lower=-1.309 upper=0 effort=0 velocity=0
- joint thumb_aa_joint: limit lower=-0.785 upper=0.785 effort=0 velocity=0 -> lower=-1.309 upper=0.785 effort=0 velocity=0
- joint thumb_distal_joint: limit lower=-0.698 upper=0 effort=0 velocity=0 -> lower=-1.309 upper=0 effort=0 velocity=0
- joint thumb_metacarpal_joint: limit lower=-0.698 upper=0 effort=0 velocity=0 -> lower=-0.262 upper=0 effort=0 velocity=0
- joint thumb_proximal_joint: limit lower=-0.698 upper=0 effort=0 velocity=0 -> lower=-1.309 upper=0 effort=0 velocity=0; mimic joint=thumb_metacarpal_joint multiplier=1 offset=0 -> joint=thumb_metacarpal_joint multiplier=5 offset=0
