Commit message: Create trajectory between current joint state and desired

File: src/roborscht_description/urdf/roborscht_v3.urdf (robot description, URDF)
Before this commit: robot roborscht_v3, 22 links, 21 joints
Joints:
- joint index_distal_joint: limit lower=0 upper=0.698 effort=0 velocity=0 -> lower=0 upper=0.5236 effort=0 velocity=0
- joint index_middle_joint: limit lower=0 upper=0.698 effort=0 velocity=0 -> lower=0 upper=0.5236 effort=0 velocity=0
- joint index_proximal_joint: limit lower=0 upper=0.698 effort=0 velocity=0 -> lower=0 upper=0.5236 effort=0 velocity=0
- joint little_distal_joint: limit lower=0 upper=0.698 effort=0 velocity=0 -> lower=0 upper=0.5236 effort=0 velocity=0
- joint little_middle_joint: limit lower=0 upper=0.698 effort=0 velocity=0 -> lower=0 upper=0.5236 effort=0 velocity=0
- joint little_proximal_joint: limit lower=0 upper=0.698 effort=0 velocity=0 -> lower=0 upper=0.5236 effort=0 velocity=0
- joint middle_distal_joint: limit lower=0 upper=0.698 effort=0 velocity=0 -> lower=0 upper=0.5236 effort=0 velocity=0
- joint middle_middle_joint: limit lower=0 upper=0.698 effort=0 velocity=0 -> lower=0 upper=0.5236 effort=0 velocity=0
- joint middle_proximal_joint: limit lower=0 upper=0.698 effort=0 velocity=0 -> lower=0 upper=0.5236 effort=0 velocity=0
- joint ring_distal_joint: limit lower=0 upper=0.698 effort=0 velocity=0 -> lower=0 upper=0.5236 effort=0 velocity=0
- joint ring_middle_joint: limit lower=0 upper=0.698 effort=0 velocity=0 -> lower=0 upper=0.5236 effort=0 velocity=0
- joint ring_proximal_joint: limit lower=0 upper=0.698 effort=0 velocity=0 -> lower=0 upper=0.5236 effort=0 velocity=0
- joint thumb_distal_joint: limit lower=0 upper=0.698 effort=0 velocity=0 -> lower=0 upper=0.5236 effort=0 velocity=0
- joint thumb_metacarpal_joint: limit lower=0 upper=0.698 effort=0 velocity=0 -> lower=0 upper=0.5236 effort=0 velocity=0
- joint thumb_proximal_joint: limit lower=0 upper=0.698 effort=0 velocity=0 -> lower=0 upper=0.5236 effort=0 velocity=0
